File: DS1339 RTC Module.brd (EAGLE design)
At the start: 24.1 x 18.5 mm, 12 parts, among them U1 DS1339AU, Y1 ECS-.327-6-17X-TR

Commit message: Added BOM and values
Parts:
- R1, R2: value (none) -> 4.7k
- R3: value (none) -> 10k
Connections:
- removed net N$8: J1.5
Changed lines of the file:
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@@
 <attribute name="VALUE" x="4.572" y="1.905" size="0.6096" layer="27" font="vector" ratio="20" rot="R90"/>
 </element>
-<element name="R1" library="SparkFun-Resistors" package="0805" value=" " x="20.32" y="8.255" smashed="yes">
+<element name="R1" library="SparkFun-Resistors" package="0805" value="4.7k" x="20.32" y="8.255" smashed="yes">
 <attribute name="NAME" x="20.32" y="9.144" size="0.8128" layer="25" font="vector" align="bottom-center"/>
 <attribute name="PROD_ID" value=" " x="35.56" y="-24.765" size="1.778" layer="27" display="off"/>
 <attribute name="VALUE" x="20.32" y="7.366" size="0.6096" layer="27" font="vector" ratio="20" align="top-center"/>
 </element>
-<element name="R2" library="SparkFun-Resistors" package="0805" value=" " x="20.32" y="5.715" smashed="yes">
+<element name="R2" library="SparkFun-Resistors" package="0805" value="4.7k" x="20.32" y="5.715" smashed="yes">
 <attribute name="NAME" x="20.32" y="6.604" size="0.8128" layer="25" font="vector" align="bottom-center"/>
 <attribute name="PROD_ID" value=" " x="39.37" y="-27.305" size="1.778" layer="27" display="off"/>
 <attribute name="VALUE" x="20.32" y="4.826" size="0.6096" layer="27" font="vector" ratio="20" align="top-center"/>
 </element>
-<element name="R3" library="SparkFun-Resistors" package="0805" value=" " x="20.32" y="12.065" smashed="yes" rot="R270">
+<element name="R3" library="SparkFun-Resistors" package="0805" value="10k" x="20.32" y="12.065" smashed="yes" rot="R270">
 <attribute name="NAME" x="21.209" y="12.065" size="0.8128" layer="25" font="vector" rot="R270" align="bottom-center"/>
 <attribute name="PROD_ID" value=" " x="-12.7" y="-10.795" size="1.778" layer="27" rot="R270" display="off"/>
@@
 <contactref element="J1" pad="6"/>
 </signal>
-<signal name="N$8">
-<contactref element="J1" pad="5"/>
-</signal>
 <signal name="INT">
